File: hardware/pcb/ups_main.sch (EAGLE design)
At the start: 83 parts, among them IC1 LTC4416EMS-1#PBF, IC2 LTC4079EDD#TRPBF, IC3 STM32F405RGT6, IC4 TPS613782QWRTERQ1, IC5 MCS1802GS-20-Z, J1 694106301002, J2 694106301002, J3 694106301002, Q1 IPD068P03L3GATMA1, Q2 IPD068P03L3GATMA1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

Commit message: update schem
Parts:
- R12: value 158k -> 280k
- R13: value 158k -> 20k
Changed lines of the file:
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@@
 <part name="GND4" library="SparkFun-PowerSymbols" deviceset="GND" device=""/>
 <part name="IC4" library="TPS613783QWRTERQ1" library_urn="urn:adsk.eagle:library:45181284" deviceset="TPS613783QWRTERQ1" device="" package3d_urn="urn:adsk.eagle:package:45181287/2" value="TPS613782QWRTERQ1"/>
-<part name="R12" library="rcl" library_urn="urn:adsk.eagle:library:334" deviceset="R-EU_" device="R0603" package3d_urn="urn:adsk.eagle:package:23555/3" value="158k"/>
-<part name="R13" library="rcl" library_urn="urn:adsk.eagle:library:334" deviceset="R-EU_" device="R0603" package3d_urn="urn:adsk.eagle:package:23555/3" value="158k"/>
+<part name="R12" library="rcl" library_urn="urn:adsk.eagle:library:334" deviceset="R-EU_" device="R0603" package3d_urn="urn:adsk.eagle:package:23555/3" value="280k"/>
+<part name="R13" library="rcl" library_urn="urn:adsk.eagle:library:334" deviceset="R-EU_" device="R0603" package3d_urn="urn:adsk.eagle:package:23555/3" value="20k"/>
 <part name="GND5" library="SparkFun-PowerSymbols" deviceset="GND" device=""/>
 <part name="R14" library="rcl" library_urn="urn:adsk.eagle:library:334" deviceset="R-EU_" device="R0603" package3d_urn="urn:adsk.eagle:package:23555/3" value="80.6k"/>

Commit message: fix errors in schem/layout
Parts:
- added C24: T491D226M035AT, T491D226M035AT:T491D226M035AT
- added C25: 1uF, rcl:C-EUC0603K
- added C26: 22uF, rcl:C-EUC0603K
Connections:
- removed net N$29: C10.2, IC4.VCC
- new net N$37: C10.2, IC4.EN, IC4.VCC
- net +12V: now also C24.+
- net GND: now also C24.-, C25.1, C26.1
- net VBAT1: now also C25.2
- net VBAT2: now also C26.2; no longer IC4.EN
Other:
- moved on the sheet: C8, L1
Changed lines of the file:
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@@
 <part name="+3V10" library="supply1" library_urn="urn:adsk.eagle:library:371" deviceset="+3V3" device=""/>
 <part name="+3V11" library="supply1" library_urn="urn:adsk.eagle:library:371" deviceset="+3V3" device=""/>
+<part name="C24" library="T491D226M035AT" library_urn="urn:adsk.eagle:library:41356059" deviceset="T491D226M035AT" device="" package3d_urn="urn:adsk.eagle:package:41356062/3"/>
+<part name="GND12" library="SparkFun-PowerSymbols" deviceset="GND" device=""/>
+<part name="C25" library="rcl" library_urn="urn:adsk.eagle:library:334" deviceset="C-EU" device="C0603K" package3d_urn="urn:adsk.eagle:package:23680/2" value="1uF"/>
+<part name="GND34" library="SparkFun-PowerSymbols" deviceset="GND" device=""/>
+<part name="GND51" library="SparkFun-PowerSymbols" deviceset="GND" device=""/>
+<part name="C26" library="rcl" library_urn="urn:adsk.eagle:library:334" deviceset="C-EU" device="C0603K" package3d_urn="urn:adsk.eagle:package:23680/2" value="22uF"/>
 </parts>
 <sheets>
@@
 <attribute name="VALUE" x="132.461" y="224.536" size="1.778" layer="96" rot="R270"/>
 </instance>
-<instance part="C8" gate="G$1" x="45.72" y="241.3" smashed="yes" rot="R270">
-<attribute name="NAME" x="42.164" y="236.601" size="1.778" layer="95"/>
-<attribute name="VALUE" x="37.084" y="239.141" size="1.778" layer="96"/>
+<instance part="C8" gate="G$1" x="53.34" y="241.3" smashed="yes" rot="R270">
+<attribute name="NAME" x="49.784" y="236.601" size="1.778" layer="95"/>
+<attribute name="VALUE" x="44.704" y="239.141" size="1.778" layer="96"/>
 </instance>
 <instance part="R16" gate="G$1" x="116.84" y="210.82" smashed="yes" rot="R90">
@@
 <attribute name="VALUE" x="117.475" y="272.288" size="1.778" layer="96" rot="R90"/>
 </instance>
-<instance part="L1" gate="G$1" x="35.56" y="243.84" smashed="yes" rot="R90">
-<attribute name="NAME" x="29.21" y="260.35" size="1.778" layer="95" rot="R90" align="center-left"/>
-<attribute name="VALUE" x="31.75" y="260.35" size="1.778" layer="96" rot="R90" align="center-left"/>
+<instance part="L1" gate="G$1" x="43.18" y="243.84" smashed="yes" rot="R90">
+<attribute name="NAME" x="36.83" y="260.35" size="1.778" layer="95" rot="R90" align="center-left"/>
+<attribute name="VALUE" x="39.37" y="260.35" size="1.778" layer="96" rot="R90" align="center-left"/>
 </instance>
 <instance part="GND35" gate="1" x="66.04" y="200.66" smashed="yes">
@@
 <instance part="+3V11" gate="G$1" x="111.76" y="297.18" smashed="yes">
 <attribute name="VALUE" x="114.3" y="297.18" size="1.778" layer="96" rot="R90"/>
+</instance>
+<instance part="C24" gate="G$1" x="-27.94" y="312.42" smashed="yes" rot="R270">
+<attribute name="NAME" x="-21.59" y="303.53" size="1.778" layer="95" rot="R270" align="center-left"/>
+<attribute name="VALUE" x="-24.13" y="303.53" size="1.778" layer="96" rot="R270" align="center-left"/>
+</instance>
+<instance part="GND12" gate="1" x="-27.94" y="289.56" smashed="yes">
+<attribute name="VALUE" x="-27.94" y="289.306" size="1.778" layer="96" font="vector" align="top-center"/>
+</instance>
+<instance part="C25" gate="G$1" x="25.4" y="238.76" smashed="yes" rot="R180">
+<attribute name="NAME" x="20.701" y="242.316" size="1.778" layer="95" rot="R270"/>
+<attribute name="VALUE" x="23.241" y="247.396" size="1.778" layer="96" rot="R270"/>
+</instance>
+<instance part="GND34" gate="1" x="25.4" y="213.36" smashed="yes">
+<attribute name="VALUE" x="25.4" y="213.106" size="1.778" layer="96" font="vector" align="top-center"/>
+</instance>
+<instance part="GND51" gate="1" x="35.56" y="213.36" smashed="yes">
+<attribute name="VALUE" x="35.56" y="213.106" size="1.778" layer="96" font="vector" align="top-center"/>
+</instance>
+<instance part="C26" gate="G$1" x="35.56" y="238.76" smashed="yes" rot="R180">
+<attribute name="NAME" x="30.861" y="242.316" size="1.778" layer="95" rot="R270"/>
+<attribute name="VALUE" x="33.401" y="247.396" size="1.778" layer="96" rot="R270"/>
 </instance>
 </instances>
@@
 <pinref part="GND52" gate="1" pin="GND"/>
 </segment>
+<segment>
+<pinref part="C24" gate="G$1" pin="-"/>
+<wire x1="-27.94" y1="299.72" x2="-27.94" y2="292.1" width="0.1524" layer="91"/>
+<pinref part="GND12" gate="1" pin="GND"/>
+</segment>
+<segment>
+<pinref part="C25" gate="G$1" pin="1"/>
+<wire x1="25.4" y1="236.22" x2="25.4" y2="215.9" width="0.1524" layer="91"/>
+<pinref part="GND34" gate="1" pin="GND"/>
+</segment>
+<segment>
+<wire x1="35.56" y1="236.22" x2="35.56" y2="215.9" width="0.1524" layer="91"/>
+<pinref part="GND51" gate="1" pin="GND"/>
+<pinref part="C26" gate="G$1" pin="1"/>
+</segment>
 </net>
 <net name="+3V3" class="0">
@@
 <junction x="20.32" y="246.38"/>
 <label x="25.4" y="251.46" size="1.27" layer="95" rot="R90" xref="yes"/>
+<pinref part="C25" gate="G$1" pin="2"/>
+<wire x1="25.4" y1="243.84" x2="25.4" y2="246.38" width="0.1524" layer="91"/>
+<junction x="25.4" y="246.38"/>
 </segment>
 <segment>
@@
 <wire x1="-40.64" y1="314.96" x2="-40.64" y2="317.5" width="0.1524" layer="91"/>
 <pinref part="P+8" gate="1" pin="+12V"/>
+<pinref part="C24" gate="G$1" pin="+"/>
+<wire x1="-27.94" y1="312.42" x2="-27.94" y2="314.96" width="0.1524" layer="91"/>
+<wire x1="-27.94" y1="314.96" x2="-40.64" y2="314.96" width="0.1524" layer="91"/>
+<junction x="-40.64" y="314.96"/>
 </segment>
 </net>
@@
 <segment>
 <pinref part="IC4" gate="G$1" pin="BST"/>
-<wire x1="71.12" y1="241.3" x2="48.26" y2="241.3" width="0.1524" layer="91"/>
+<wire x1="71.12" y1="241.3" x2="55.88" y2="241.3" width="0.1524" layer="91"/>
 <pinref part="C8" gate="G$1" pin="1"/>
 </segment>
@@
 <segment>
 <pinref part="IC4" gate="G$1" pin="SW_2"/>
-<wire x1="71.12" y1="236.22" x2="35.56" y2="236.22" width="0.1524" layer="91"/>
-<wire x1="35.56" y1="236.22" x2="35.56" y2="241.3" width="0.1524" layer="91"/>
+<wire x1="71.12" y1="236.22" x2="43.18" y2="236.22" width="0.1524" layer="91"/>
+<wire x1="43.18" y1="236.22" x2="43.18" y2="241.3" width="0.1524" layer="91"/>
 <pinref part="IC4" gate="G$1" pin="SW_1"/>
 <wire x1="71.12" y1="238.76" x2="71.12" y2="236.22" width="0.1524" layer="91"/>
 <junction x="71.12" y="236.22"/>
 <pinref part="C8" gate="G$1" pin="2"/>
-<wire x1="40.64" y1="241.3" x2="35.56" y2="241.3" width="0.1524" layer="91"/>
-<wire x1="35.56" y1="241.3" x2="35.56" y2="243.84" width="0.1524" layer="91"/>
-<junction x="35.56" y="241.3"/>
+<wire x1="48.26" y1="241.3" x2="43.18" y2="241.3" width="0.1524" layer="91"/>
+<wire x1="43.18" y1="241.3" x2="43.18" y2="243.84" width="0.1524" layer="91"/>
+<junction x="43.18" y="241.3"/>
 <pinref part="L1" gate="G$1" pin="1"/>
 </segment>
@@
 </segment>
 </net>
-<net name="N$29" class="0">
-<segment>
-<pinref part="C10" gate="G$1" pin="2"/>
-<pinref part="IC4" gate="G$1" pin="VCC"/>
-<wire x1="83.82" y1="210.82" x2="83.82" y2="213.36" width="0.1524" layer="91"/>
-</segment>
-</net>
 <net name="N$4" class="0">
 <segment>
@@
 <net name="VBAT2" class="0">
 <segment>
-<pinref part="IC4" gate="G$1" pin="EN"/>
-<wire x1="86.36" y1="259.08" x2="86.36" y2="266.7" width="0.1524" layer="91"/>
-<wire x1="86.36" y1="266.7" x2="60.96" y2="266.7" width="0.1524" layer="91"/>
 <pinref part="IC4" gate="G$1" pin="VIN"/>
 <wire x1="71.12" y1="243.84" x2="60.96" y2="243.84" width="0.1524" layer="91"/>
 <wire x1="60.96" y1="243.84" x2="60.96" y2="266.7" width="0.1524" layer="91"/>
-<wire x1="60.96" y1="266.7" x2="35.56" y2="266.7" width="0.1524" layer="91"/>
-<junction x="60.96" y="266.7"/>
+<wire x1="60.96" y1="266.7" x2="43.18" y2="266.7" width="0.1524" layer="91"/>
+<wire x1="43.18" y1="266.7" x2="35.56" y2="266.7" width="0.1524" layer="91"/>
 <wire x1="35.56" y1="266.7" x2="35.56" y2="271.78" width="0.1524" layer="91"/>
 <label x="35.56" y="271.78" size="1.27" layer="95" rot="R90" xref="yes"/>
-<wire x1="35.56" y1="266.7" x2="35.56" y2="264.16" width="0.1524" layer="91"/>
 <junction x="35.56" y="266.7"/>
 <pinref part="L1" gate="G$1" pin="2"/>
+<wire x1="43.18" y1="264.16" x2="43.18" y2="266.7" width="0.1524" layer="91"/>
+<junction x="43.18" y="266.7"/>
+<wire x1="35.56" y1="266.7" x2="35.56" y2="243.84" width="0.1524" layer="91"/>
+<pinref part="C26" gate="G$1" pin="2"/>
 </segment>
 <segment>
@@
 </segment>
 </net>
+<net name="N$37" class="0">
+<segment>
+<pinref part="IC4" gate="G$1" pin="EN"/>
+<wire x1="86.36" y1="259.08" x2="86.36" y2="266.7" width="0.1524" layer="91"/>
+<wire x1="86.36" y1="266.7" x2="68.58" y2="266.7" width="0.1524" layer="91"/>
+<wire x1="68.58" y1="266.7" x2="68.58" y2="210.82" width="0.1524" layer="91"/>
+<pinref part="C10" gate="G$1" pin="2"/>
+<pinref part="IC4" gate="G$1" pin="VCC"/>
+<wire x1="83.82" y1="210.82" x2="83.82" y2="213.36" width="0.1524" layer="91"/>
+<wire x1="68.58" y1="210.82" x2="83.82" y2="210.82" width="0.1524" layer="91"/>
+<junction x="83.82" y="210.82"/>
+</segment>
+</net>

Commit message: fix pgood led
Connections:
- net +3V3: no longer R17.2
- net GND: now also PGOOD.C
- net N$13: now also R17.2; no longer PGOOD.C
Other:
- moved on the sheet: PGOOD, R17
Changed lines of the file:
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@@
 <part name="P+4" library="supply1" library_urn="urn:adsk.eagle:library:371" deviceset="VCC" device=""/>
 <part name="+3V10" library="supply1" library_urn="urn:adsk.eagle:library:371" deviceset="+3V3" device=""/>
-<part name="+3V11" library="supply1" library_urn="urn:adsk.eagle:library:371" deviceset="+3V3" device=""/>
 <part name="C24" library="T491D226M035AT" library_urn="urn:adsk.eagle:library:41356059" deviceset="T491D226M035AT" device="" package3d_urn="urn:adsk.eagle:package:41356062/3"/>
 <part name="GND12" library="SparkFun-PowerSymbols" deviceset="GND" device=""/>
@@
 <part name="GND51" library="SparkFun-PowerSymbols" deviceset="GND" device=""/>
 <part name="C26" library="rcl" library_urn="urn:adsk.eagle:library:334" deviceset="C-EU" device="C0603K" package3d_urn="urn:adsk.eagle:package:23680/2" value="22uF"/>
+<part name="GND53" library="SparkFun-PowerSymbols" deviceset="GND" device=""/>
 </parts>
 <sheets>
@@
 <attribute name="VALUE" x="115.062" y="212.09" size="1.778" layer="96" rot="R90"/>
 </instance>
-<instance part="R17" gate="G$1" x="111.76" y="287.02" smashed="yes" rot="R90">
-<attribute name="NAME" x="110.2614" y="283.21" size="1.778" layer="95" rot="R90"/>
-<attribute name="VALUE" x="109.982" y="288.29" size="1.778" layer="96" rot="R90"/>
+<instance part="R17" gate="G$1" x="111.76" y="223.52" smashed="yes" rot="R90">
+<attribute name="NAME" x="110.2614" y="219.71" size="1.778" layer="95" rot="R90"/>
+<attribute name="VALUE" x="109.982" y="224.79" size="1.778" layer="96" rot="R90"/>
 </instance>
 <instance part="C9" gate="G$1" x="104.14" y="220.98" smashed="yes" rot="R180">
@@
 <attribute name="VALUE" x="13.335" y="249.428" size="1.778" layer="96" rot="R90"/>
 </instance>
-<instance part="PGOOD" gate="G$1" x="111.76" y="276.86" smashed="yes">
-<attribute name="NAME" x="107.696" y="274.828" size="1.778" layer="95" rot="R90"/>
-<attribute name="VALUE" x="117.475" y="272.288" size="1.778" layer="96" rot="R90"/>
+<instance part="PGOOD" gate="G$1" x="111.76" y="213.36" smashed="yes">
+<attribute name="NAME" x="107.696" y="211.328" size="1.778" layer="95" rot="R90"/>
+<attribute name="VALUE" x="117.475" y="208.788" size="1.778" layer="96" rot="R90"/>
 </instance>
 <instance part="L1" gate="G$1" x="43.18" y="243.84" smashed="yes" rot="R90">
@@
 <attribute name="VALUE" x="10.16" y="274.32" size="1.778" layer="96" rot="R90"/>
 </instance>
-<instance part="+3V11" gate="G$1" x="111.76" y="297.18" smashed="yes">
-<attribute name="VALUE" x="114.3" y="297.18" size="1.778" layer="96" rot="R90"/>
-</instance>
 <instance part="C24" gate="G$1" x="-27.94" y="312.42" smashed="yes" rot="R270">
 <attribute name="NAME" x="-21.59" y="303.53" size="1.778" layer="95" rot="R270" align="center-left"/>
@@
 <attribute name="NAME" x="30.861" y="242.316" size="1.778" layer="95" rot="R270"/>
 <attribute name="VALUE" x="33.401" y="247.396" size="1.778" layer="96" rot="R270"/>
+</instance>
+<instance part="GND53" gate="1" x="111.76" y="200.66" smashed="yes">
+<attribute name="VALUE" x="111.76" y="200.406" size="1.778" layer="96" font="vector" align="top-center"/>
 </instance>
 </instances>
@@
 <pinref part="C26" gate="G$1" pin="1"/>
 </segment>
+<segment>
+<pinref part="GND53" gate="1" pin="GND"/>
+<pinref part="PGOOD" gate="G$1" pin="C"/>
+<wire x1="111.76" y1="203.2" x2="111.76" y2="208.28" width="0.1524" layer="91"/>
+</segment>
 </net>
 <net name="+3V3" class="0">
@@
 <pinref part="R9" gate="G$1" pin="2"/>
 <wire x1="7.62" y1="271.78" x2="7.62" y2="269.24" width="0.1524" layer="91"/>
-</segment>
-<segment>
-<pinref part="+3V11" gate="G$1" pin="+3V3"/>
-<pinref part="R17" gate="G$1" pin="2"/>
-<wire x1="111.76" y1="294.64" x2="111.76" y2="292.1" width="0.1524" layer="91"/>
 </segment>
 </net>
@@
 <pinref part="IC4" gate="G$1" pin="PG"/>
 <wire x1="101.6" y1="241.3" x2="111.76" y2="241.3" width="0.1524" layer="91"/>
-<pinref part="PGOOD" gate="G$1" pin="C"/>
-<wire x1="111.76" y1="271.78" x2="111.76" y2="241.3" width="0.1524" layer="91"/>
+<pinref part="R17" gate="G$1" pin="2"/>
+<wire x1="111.76" y1="228.6" x2="111.76" y2="241.3" width="0.1524" layer="91"/>
 </segment>
 </net>
@@
 <pinref part="PGOOD" gate="G$1" pin="A"/>
 <pinref part="R17" gate="G$1" pin="1"/>
-<wire x1="111.76" y1="279.4" x2="111.76" y2="281.94" width="0.1524" layer="91"/>
-</segment>
-</net>
+<wire x1="111.76" y1="215.9" x2="111.76" y2="218.44" width="0.1524" layer="91"/>
+</segment>
+</net>
